Commit message: added the camera params file

File: urdf/pauvsi_m7_robot.urdf (robot description, URDF)
Before this commit: robot pauvsi_m7_robot, 2 links, 1 joints
Links:
- added link arm2_link; visual cylinder length=0.334 radius=0.036
- added link arm3_link; visual cylinder length=0.334 radius=0.036
- added link arm4_link; visual cylinder length=0.334 radius=0.036
- added link motor1_link; visual cylinder length=0.01 radius=0.2286
- added link motor2_link; visual cylinder length=0.01 radius=0.2286
- added link motor3_link; visual cylinder length=0.01 radius=0.2286
- added link motor4_link; visual cylinder length=0.01 radius=0.2286
- link arm1_link: geometry visual cylinder length=0.334 radius=0.036
Joints:
- added joint base_to_arm2: type fixed, parent base_link, child arm2_link, origin xyz=0.18 -0.18 0
- added joint base_to_arm3: type fixed, parent base_link, child arm3_link, origin xyz=-0.18 -0.18 0
- added joint base_to_arm4: type fixed, parent base_link, child arm4_link, origin xyz=-0.18 0.18 0
- added joint motor1_to_arm1: type fixed, parent arm1_link, child motor1_link, origin xyz=0.13 0.13 0.06
- added joint motor2_to_arm2: type fixed, parent arm2_link, child motor2_link, origin xyz=0.13 -0.13 0.06
- added joint motor3_to_arm3: type fixed, parent arm3_link, child motor3_link, origin xyz=-0.13 -0.13 0.06
- added joint motor4_to_arm4: type fixed, parent arm4_link, child motor4_link, origin xyz=-0.13 0.13 0.06
- joint base_to_arm1: origin xyz=-0.18 0.18 0 -> xyz=0.18 0.18 0
